Commit message: wip

File: quadruped_full.urdf (robot description, URDF)
Before this commit: robot robot, 14 links, 13 joints
Joints:
- joint base_joint: origin xyz=0 0 0 rpy=0 0 0 -> xyz=0 0 0.3 rpy=0 0 0

Commit message: wip

File: quadruped_full.urdf (robot description, URDF)
Before this commit: robot robot, 14 links, 13 joints
Links:
- link fl_foot: geometry collision box size=0.3 0.05 0.05; visual box size=0.45 0.05 0.05
- link fr_foot: geometry collision box size=0.3 0.05 0.05; visual box size=0.45 0.05 0.05
- link rl_foot: geometry collision box size=0.3 0.05 0.05; visual box size=0.45 0.05 0.05
- link rr_foot: geometry collision box size=0.3 0.05 0.05; visual box size=0.45 0.05 0.05
Joints:
- joint base_joint: origin xyz=0 0 0.3 rpy=0 0 0 -> xyz=0 0 0 rpy=0 0 0
- joint base_link_to_fl_hip: limit lower=-1 upper=1 effort=1000.0 velocity=0.5 -> lower=-2 upper=2 effort=1000.0 velocity=0.5
- joint base_link_to_fr_hip: limit lower=-1 upper=1 effort=1000.0 velocity=0.5 -> lower=-2 upper=2 effort=1000.0 velocity=0.5
- joint base_link_to_rl_hip: limit lower=-1 upper=1 effort=1000.0 velocity=0.5 -> lower=-2 upper=2 effort=1000.0 velocity=0.5
- joint base_link_to_rr_hip: limit lower=-1 upper=1 effort=1000.0 velocity=0.5 -> lower=-2 upper=2 effort=1000.0 velocity=0.5
- joint fl_hip_to_fl_knee: limit lower=-1 upper=1 effort=1000.0 velocity=0.5 -> lower=-2 upper=2 effort=1000.0 velocity=0.5
- joint fl_knee_to_fl_foot: limit lower=-1 upper=1 effort=1000.0 velocity=0.5 -> lower=-2 upper=2 effort=1000.0 velocity=0.5; origin xyz=0.30056379478285833 -5.551115123125783e-17 -2.465190328815662e-32 rpy=0 0 0 -> xyz=0.30000000000000004 0 5.55111512312578e-17 rpy=0 0 0
- joint fr_hip_to_fr_knee: limit lower=-1 upper=1 effort=1000.0 velocity=0.5 -> lower=-2 upper=2 effort=1000.0 velocity=0.5
- joint fr_knee_to_fr_foot: limit lower=-1 upper=1 effort=1000.0 velocity=0.5 -> lower=-2 upper=2 effort=1000.0 velocity=0.5
- joint rl_hip_to_rl_knee: limit lower=-1 upper=1 effort=1000.0 velocity=0.5 -> lower=-2 upper=2 effort=1000.0 velocity=0.5
- joint rl_knee_to_rl_foot: limit lower=-1 upper=1 effort=1000.0 velocity=0.5 -> lower=-2 upper=2 effort=1000.0 velocity=0.5
- joint rr_hip_to_rr_knee: limit lower=-1 upper=1 effort=1000.0 velocity=0.5 -> lower=-2 upper=2 effort=1000.0 velocity=0.5
- joint rr_knee_to_rr_foot: limit lower=-1 upper=1 effort=1000.0 velocity=0.5 -> lower=-2 upper=2 effort=1000.0 velocity=0.5
